File: pcb/LightBrain.kicad_sch (KiCad schematic)
At the start: 50 parts, among them J1 Wago2060, J2 Wago2060, J3 Wago2060, J5 Wago2060, Q1 AO3401A, SW1 SW_Push, SW2 SW_Push, SW3 SW_Push, U1 SN75176BDR, U2 74LVC1G34W5-7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

Commit message: Doc files, slight fixes, initial readme.md content
Other:
- title: LightBrain Chematic -> LightBrain Schematic
Changed lines of the file:
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@@
   (paper "A4")
   (title_block
-    (title "LightBrain Chematic")
+    (title "LightBrain Schematic")
     (date "2022-03-19")
     (rev "2.2")
